File: buck.kicad_sch (KiCad schematic)
At the start: 31 parts, among them Q1 PMOS, U1 ${SIM.PARAMS}, U2 ${SIM.PARAMS}, U3 ${SIM.PARAMS}, U4 ${SIM.PARAMS}, U5 ${SIM.PARAMS}, U6 ${SIM.PARAMS}

Commit message: updated files
Parts:
- removed L2: 1mH, symbol Device:L
Connections:
- net Vout: now also R1.1
Other:
- moved on the sheet: R1
Changed lines of the file:
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@@
-	(wire
-		(pts
-			(xy 64.77 176.53) (xy 64.77 181.61)
-		)
-		(stroke
-			(width 0)
-			(type default)
-		)
-	)
 	(wire
 		(pts
@@
 	(wire
 		(pts
-			(xy 64.77 165.1) (xy 64.77 168.91)
+			(xy 63.5 165.1) (xy 63.5 167.64)
 		)
 		(stroke
@@
 	(wire
 		(pts
-			(xy 64.77 189.23) (xy 64.77 195.58)
+			(xy 63.5 175.26) (xy 63.5 181.61)
 		)
 		(stroke
@@
 	(wire
 		(pts
-			(xy 64.77 165.1) (xy 50.8 165.1)
+			(xy 63.5 165.1) (xy 50.8 165.1)
 		)
 		(stroke
@@
 	)
 	(label "Vout"
-		(at 64.77 165.1 0)
+		(at 63.5 165.1 0)
 		(effects
 			(font
@@
 	)
 	(symbol
-		(lib_id "Device:L")
-		(at 64.77 172.72 0)
-		(unit 1)
-		(body_style 1)
-		(exclude_from_sim no)
-		(in_bom yes)
-		(on_board yes)
-		(in_pos_files yes)
-		(dnp no)
-		(fields_autoplaced yes)
-		(property "Reference" "L2"
-			(at 66.04 171.4499 0)
-			(show_name no)
-			(do_not_autoplace no)
-			(effects
-				(font
-					(size 1.27 1.27)
-				)
-				(justify left)
-			)
-		)
-		(property "Value" "1mH"
-			(at 66.04 173.9899 0)
-			(show_name no)
-			(do_not_autoplace no)
-			(effects
-				(font
-					(size 1.27 1.27)
-				)
-				(justify left)
-			)
-		)
-		(property "Footprint" ""
-			(at 64.77 172.72 0)
-			(hide yes)
-			(show_name no)
-			(do_not_autoplace no)
-			(effects
-				(font
-					(size 1.27 1.27)
-				)
-			)
-		)
-		(property "Datasheet" ""
-			(at 64.77 172.72 0)
-			(hide yes)
-			(show_name no)
-			(do_not_autoplace no)
-			(effects
-				(font
-					(size 1.27 1.27)
-				)
-			)
-		)
-		(property "Description" "Inductor"
-			(at 64.77 172.72 0)
-			(hide yes)
-			(show_name no)
-			(do_not_autoplace no)
-			(effects
-				(font
-					(size 1.27 1.27)
-				)
-			)
-		)
-		(pin "2"
-		)
-		(pin "1"
-		)
-		(instances
-			(project "buck"
-				(path "/7191e9ae-ac69-4d50-90dd-2471411688c3"
-					(reference "L2")
-					(unit 1)
-				)
-			)
-		)
-	)
-	(symbol
 		(lib_id "Simulation_SPICE:0")
 		(at 175.26 111.76 0)
@@
 	(symbol
 		(lib_id "Simulation_SPICE:0")
-		(at 64.77 195.58 0)
+		(at 63.5 181.61 0)
 		(unit 1)
 		(body_style 1)
@@
 		(in_pos_files yes)
 		(dnp no)
-		(fields_autoplaced yes)
 		(property "Reference" "#GND06"
-			(at 64.77 200.66 0)
+			(at 63.5 186.69 0)
 			(hide yes)
 			(show_name no)
@@
 		)
 		(property "Value" "0"
-			(at 64.77 193.04 0)
+			(at 63.5 179.07 0)
 			(show_name no)
 			(do_not_autoplace no)
@@
 		)
 		(property "Footprint" ""
-			(at 64.77 195.58 0)
+			(at 63.5 181.61 0)
 			(hide yes)
 			(show_name no)
@@
 		)
 		(property "Datasheet" "https://ngspice.sourceforge.io/docs/ngspice-html-manual/manual.xhtml#subsec_Circuit_elements__device"
-			(at 64.77 205.74 0)
+			(at 63.5 191.77 0)
 			(hide yes)
 			(show_name no)
@@
 		)
 		(property "Description" "0V reference potential for simulation"
-			(at 64.77 203.2 0)
+			(at 63.5 189.23 0)
 			(hide yes)
 			(show_name no)
@@
 	(symbol
 		(lib_id "Device:R")
-		(at 64.77 185.42 0)
+		(at 63.5 171.45 0)
 		(unit 1)
 		(body_style 1)
@@
 		(fields_autoplaced yes)
 		(property "Reference" "R1"
-			(at 67.31 184.1499 0)
+			(at 66.04 170.1799 0)
 			(show_name no)
 			(do_not_autoplace no)
@@
 		)
 		(property "Value" "5k"
-			(at 67.31 186.6899 0)
+			(at 66.04 172.7199 0)
 			(show_name no)
 			(do_not_autoplace no)
@@
 		)
 		(property "Footprint" ""
-			(at 62.992 185.42 90)
+			(at 61.722 171.45 90)
 			(hide yes)
 			(show_name no)
@@
 		)
 		(property "Datasheet" ""
-			(at 64.77 185.42 0)
+			(at 63.5 171.45 0)
 			(hide yes)
 			(show_name no)
@@
 		)
 		(property "Description" "Resistor"
-			(at 64.77 185.42 0)
-			(hide yes)
-			(show_name no)
+			(at 63.5 171.45 0)
+			(hide yes)
+			(show_name no)
